File: T1200_PSU.kicad_pcb (KiCad board)
At the start: 2 copper layers, 144 x 58.5 mm, 41 parts, among them J1 Data, SW1 Power Switch, T1 Rev 0.1, T2 Toshiba T1200 PSU, T3 https://github.com/BasicCode, U1 LM337L_TO92, U2 LT1614CMS8-PBF, U3 K7805-2000R3, U4 K7805-2000R3

Commit message: revision 1.0
Parts:
- removed RLA1: TMV1212S, TMH1212S:TMH1212S
- added PS1: TMV_1212S, TMV1212:CONV_TMV_1212S, F.Cu at (129.5, 40.5)
- added R4: 10K, Resistor_SMD:R_1206_3216Metric, F.Cu at (141.0, 40.5)
- C2: footprint Capacitor_SMD:C_1206_3216Metric -> Capacitor_SMD:C_0805_2012Metric
- SW1: value Power Switch -> SW_SPDT; footprint TerminalBlock:TerminalBlock_Altech_AK300-3_P5.00mm -> switch:switch
- T1: value Rev 0.1 -> Rev 1.0
- moved R5 8.92 mm to (47.5, 37.5), turned to 90 degrees
- moved SW1 5.10 mm to (23.0, 52.5), turned to -90 degrees
- moved R1 1.38 mm to (51.5, 37.5)
- moved R2 1.38 mm to (54.0, 37.5)
- moved PJ1 1.00 mm to (25.0, 37.5)
Connections:
- R1 pad 1: GND -> Net-(R1-Pad1)
- R1 pad 2: Net-(R1-Pad2) -> -22V
- R2 pad 1: GND -> Net-(R1-Pad1)
- R2 pad 2: Net-(R1-Pad2) -> -22V
- R5 pad 1: Net-(R1-Pad2) -> GND
- R5 pad 2: -22V -> Net-(R1-Pad1)
- SW1 pad 1: Net-(PJ1-Pad1) -> unconnected-(SW1-Pad1)
- SW1 pad 2: Net-(F1-Pad1) -> Net-(PJ1-Pad1)
- SW1 pad 3: (no net) -> Net-(F1-Pad1)
- U2 pad 1: Net-(R1-Pad2) -> Net-(R1-Pad1)
Routing:
- net GND: track 302.6 -> 231.7 mm
- net Net-(R1-Pad2): track 19.1 -> 0.00 mm
- net Net-(R1-Pad1): track 0.00 -> 10.9 mm
- net VCC: track 148.4 -> 140.3 mm
- net +12V: track 191.5 -> 198.0 mm
- net Net-(F1-Pad1): track 7.58 -> 11.6 mm
- net Net-(PJ1-Pad1): track 23.3 -> 19.8 mm
- net -22V: track 107.4 -> 110.3 mm
Other:
- board text added: "LCD -22V"
- board text removed: "LCD, Modem -22V"

Commit message: update documentation
Parts:
- PJ6: value System Logic & FDD Power -> CPU Power
Changed lines of the file:
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@@
       (effects (font (size 1 1) (thickness 0.15)))
     )
-    (fp_line (start -9.75 3.05) (end -9.75 -3.05) (layer "F.SilkS") (width 0.127))
     (fp_line (start 9.75 3.05) (end 9.75 -3.05) (layer "F.SilkS") (width 0.127))
     (fp_line (start 9.75 3.05) (end -9.75 3.05) (layer "F.SilkS") (width 0.127))
     (fp_line (start 9.75 -3.05) (end -9.75 -3.05) (layer "F.SilkS") (width 0.127))
+    (fp_line (start -9.75 3.05) (end -9.75 -3.05) (layer "F.SilkS") (width 0.127))
     (fp_circle (center -10.438 -1.675) (end -10.338 -1.675) (layer "F.SilkS") (width 0.2) (fill none))
     (fp_line (start -10 3.3) (end -10 -3.3) (layer "F.CrtYd") (width 0.05))
+    (fp_line (start 10 -3.3) (end -10 -3.3) (layer "F.CrtYd") (width 0.05))
     (fp_line (start 10 3.3) (end -10 3.3) (layer "F.CrtYd") (width 0.05))
     (fp_line (start 10 3.3) (end 10 -3.3) (layer "F.CrtYd") (width 0.05))
-    (fp_line (start 10 -3.3) (end -10 -3.3) (layer "F.CrtYd") (width 0.05))
+    (fp_line (start 9.75 3.05) (end 9.75 -3.05) (layer "F.Fab") (width 0.127))
+    (fp_line (start -9.75 3.05) (end -9.75 -3.05) (layer "F.Fab") (width 0.127))
+    (fp_line (start 9.75 -3.05) (end -9.75 -3.05) (layer "F.Fab") (width 0.127))
     (fp_line (start 9.75 3.05) (end -9.75 3.05) (layer "F.Fab") (width 0.127))
-    (fp_line (start 9.75 3.05) (end 9.75 -3.05) (layer "F.Fab") (width 0.127))
-    (fp_line (start 9.75 -3.05) (end -9.75 -3.05) (layer "F.Fab") (width 0.127))
-    (fp_line (start -9.75 3.05) (end -9.75 -3.05) (layer "F.Fab") (width 0.127))
     (fp_circle (center -10.438 -1.675) (end -10.338 -1.675) (layer "F.Fab") (width 0.2) (fill none))
     (pad "1" thru_hole rect (at -7.65 -1.675) (size 1.218 1.218) (drill 0.71) (layers *.Cu *.Mask)
@@
       (effects (font (size 1 1) (thickness 0.15)))
     )
-    (fp_text value "System Logic & FDD Power" (at 4.5 1.275 180) (layer "F.SilkS")
+    (fp_text value "CPU Power" (at 4.5 1.275 180) (layer "F.SilkS")
       (effects (font (size 1 1) (thickness 0.15)))
     )
