File: T1200_PSU.kicad_sch (KiCad schematic)
At the start: 41 parts, among them J1 Data, SW1 Power Switch, T1 Rev 0.1, T2 Toshiba T1200 PSU, T3 https://github.com/BasicCode, U1 LM337L_TO92, U2 LT1614CMS8-PBF, U3 K7805-2000R3, U4 K7805-2000R3

Commit message: revision 1.0
Parts:
- removed RLA1: TMV1212S, TMH1212S:TMH1212S, symbol TMS1212S:TMH1212S
- removed SW1: Power Switch, TerminalBlock:TerminalBlock_Altech_AK300-3_P5.00mm, symbol Switch:SW_SPST
- added PS1: TMV_1212S, CONV_TMV_1212S, symbol TMV1212S:TMV_1212S
- added R4: 10K, Resistor_SMD:R_1206_3216Metric, symbol Device:R
- added SW1: (no value), symbol Switch:SW_SPDT
- C2: footprint Capacitor_SMD:C_1206_3216Metric -> Capacitor_SMD:C_0805_2012Metric
- T1: value Rev 0.1 -> Rev 1.0
Connections:
- net +12V: now also PS1.7 (+VOUT), R4.1
- net -22V: now also R1.2, R2.2; no longer R5.2
- net GND: now also R5.1, PS1.2 (-VIN_(GND)), PS1.5 (-VOUT), R4.2; no longer R1.1, R2.1
- net VCC: now also PS1.1 (+VIN_(VCC))
- net at PJ1.1: now also SW1.2 (B)
- net at F1.1: now also SW1.3 (C)
- new net: R1.1, R2.1, R5.2, U2.1 (NFB)
Other:
- moved on the sheet: R1, R2, R5

Commit message: update documentation
Parts:
- PJ6: value System Logic & FDD Power -> (none)
- SW1: value (none) -> SW_SPDT; footprint (none) -> switch:switch
Other:
- note added: "CPU Power"
- note removed: "System Logic & FDD Power"
Changed lines of the file:
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@@
     (effects (font (size 2 2)) (justify left bottom))
   )
-  (text "System Logic & FDD Power" (at 17.78 132.08 0)
+  (text "CPU Power" (at 17.78 132.08 0)
     (effects (font (size 2 2)) (justify left bottom))
   )
@@
     (in_bom yes) (on_board yes) (fields_autoplaced)
     (property "Reference" "SW1" (id 0) (at 39.37 19.05 0))
-    (property "Value" "" (id 1) (at 39.37 21.59 0))
-    (property "Footprint" "" (id 2) (at 39.37 26.67 0)
+    (property "Value" "SW_SPDT" (id 1) (at 39.37 21.59 0))
+    (property "Footprint" "switch:switch" (id 2) (at 39.37 26.67 0)
       (effects (font (size 1.27 1.27)) hide)
     )
@@
     (in_bom yes) (on_board yes)
     (property "Reference" "PJ6" (id 0) (at 25.4 142.24 0))
-    (property "Value" "System Logic & FDD Power" (id 1) (at 34.29 134.62 0))
+    (property "Value" "" (id 1) (at 34.29 134.62 0))
     (property "Footprint" "Connector_PinHeader_2.54mm:PinHeader_1x02_P2.54mm_Vertical" (id 2) (at 25.4 137.16 0)
       (effects (font (size 1.27 1.27)) hide)
@@
     )
     (path "/d3d5faca-72bb-4ac2-bf9a-ed896c233789"
-      (reference "PJ6") (unit 1) (value "System Logic & FDD Power") (footprint "Connector_PinHeader_2.54mm:PinHeader_1x02_P2.54mm_Vertical")
+      (reference "PJ6") (unit 1) (value "CPU Power") (footprint "Connector_PinHeader_2.54mm:PinHeader_1x02_P2.54mm_Vertical")
     )
     (path "/69d154a6-c899-4967-9ff6-baac07f9ffa5"
